File: pcb/variants/pogo-magnetic/Symm60HE-Mag-Left-Half.kicad_pcb (KiCad board)
At the start: 2 copper layers, 158.9 x 107.8 mm, 115 parts

Commit message: Rebuild the magnetic variant around SUNMON 903-00081
Replaces the invented MAGPOGO-2x6-P254 interface drawing with a real part:
SUNMON 903-00081 / 904-00080 (MC142-09R), nine contacts in two staggered rows
on 1.50 mm pitch with 1.25 mm between rows, 1.20 mm contacts, 0.50 mm DIP
tails, and N52 magnets internal to the housing keyed N to S. Every footprint
dimension is read off the two published drawings.

Nine contacts is the link's functional minimum -- four ADC channels, three mux
selects, +3V3A and one ground -- so the twelve-way interface's four separate
grounds collapse to one and the module ties the controller ZIF's four ground
pads to that single contact.

The stagger is the hard part and it is the part's, not this attempt's:
diagonal neighbours are 1.458 mm apart with 1.25 mm pads, so nothing routes
between the contacts and every run leaves the array at its perimeter. The row
facing the ZIF drops straight to B.Cu; the other takes F.Cu over the top, down
the module side and back in above the ZIF.

Routing is not finished: 6 and 4 clearance flags on the modules, 11 on each
half. Recorded in the README along with why. Footprints, land pattern, pinout
and module outline are settled; the fanout is not.

Modules are 26 x 16 mm. docs/img/42 redraws them and docs/img/43 adds the
target breakout on the Hall PCBs.

Co-Authored-By: Claude Opus 5 <noreply@anthropic.com>
Claude-Session: https://claude.ai/code/session_01CRkZ4zVz5Mq7Fa3C5HAmii
Parts:
- PTL1: value MAGPOGO-2x6-P254-T -> 904-00080; footprint MagPogo_2x6_P254_Target -> MagPogo_9_MC142_Target
Connections:
- PTL1 pad 1: GND -> ADC_L4
- PTL1 pad 3: GND -> MUX_A2
- PTL1 pad 4: MUX_A2 -> MUX_A1
- PTL1 pad 5: MUX_A1 -> MUX_A0
- PTL1 pad 6: MUX_A0 -> ADC_L3
- PTL1 pad 7: ADC_L4 -> ADC_L1
- PTL1 pad 8: ADC_L3 -> GND
- PTL1 pad 9: ADC_L1 -> +3V3A
Routing:
- net ADC_L4: track 39.3 -> 36.5 mm, vias 4 -> 2
- net ADC_L1: track 121.0 -> 119.8 mm
- net MUX_A2: track 138.1 -> 139.2 mm
- net MUX_A1: track 138.4 -> 139.2 mm
- net +3V3A: track 850.1 -> 849.3 mm
- net MUX_A0: track 134.2 -> 133.5 mm
- net ADC_L3: track 62.2 -> 61.7 mm
