File: pcb/variants/pogo-magnetic/Symm60HE-Mag-Right-Half.kicad_pcb (KiCad board)
At the start: 2 copper layers, 158.9 x 107.8 mm, 123 parts

Commit message: Rebuild the magnetic variant around SUNMON 903-00081
Replaces the invented MAGPOGO-2x6-P254 interface drawing with a real part:
SUNMON 903-00081 / 904-00080 (MC142-09R), nine contacts in two staggered rows
on 1.50 mm pitch with 1.25 mm between rows, 1.20 mm contacts, 0.50 mm DIP
tails, and N52 magnets internal to the housing keyed N to S. Every footprint
dimension is read off the two published drawings.

Nine contacts is the link's functional minimum -- four ADC channels, three mux
selects, +3V3A and one ground -- so the twelve-way interface's four separate
grounds collapse to one and the module ties the controller ZIF's four ground
pads to that single contact.

The stagger is the hard part and it is the part's, not this attempt's:
diagonal neighbours are 1.458 mm apart with 1.25 mm pads, so nothing routes
between the contacts and every run leaves the array at its perimeter. The row
facing the ZIF drops straight to B.Cu; the other takes F.Cu over the top, down
the module side and back in above the ZIF.

Routing is not finished: 6 and 4 clearance flags on the modules, 11 on each
half. Recorded in the README along with why. Footprints, land pattern, pinout
and module outline are settled; the fanout is not.

Modules are 26 x 16 mm. docs/img/42 redraws them and docs/img/43 adds the
target breakout on the Hall PCBs.

Co-Authored-By: Claude Opus 5 <noreply@anthropic.com>
Claude-Session: https://claude.ai/code/session_01CRkZ4zVz5Mq7Fa3C5HAmii
Parts:
- PTR1: value MAGPOGO-2x6-P254-T -> 904-00080; footprint MagPogo_2x6_P254_Target -> MagPogo_9_MC142_Target
Connections:
- PTR1 pad 2: GND -> MUX_A1
- PTR1 pad 3: GND -> ADC_R1
- PTR1 pad 4: ADC_R2 -> ADC_R3
- PTR1 pad 5: ADC_R3 -> ADC_R4
- PTR1 pad 6: ADC_R4 -> MUX_A0
- PTR1 pad 7: MUX_A0 -> MUX_A2
- PTR1 pad 8: MUX_A1 -> ADC_R2
- PTR1 pad 9: MUX_A2 -> GND
Routing:
- net MUX_A1: track 136.8 -> 132.7 mm
- net MUX_A0: track 172.7 -> 169.3 mm
- net ADC_R2: track 64.9 -> 68.2 mm
- net ADC_R1: track 41.9 -> 38.7 mm
- net ADC_R3: track 101.3 -> 103.2 mm
- net +3V3A: track 957.8 -> 959.4 mm
- net ADC_R4: track 125.7 -> 127.2 mm
- net MUX_A2: track 140.8 -> 139.4 mm
