File: pcb/Symm60HE-Daughterboard.kicad_sch (KiCad schematic)
At the start: 30 parts, among them J1 TYPE-C-31-M-12, J2 FFC_12P, J3 FFC_12P, SW1 TS-1187A, SW2 TS-1187A, U1 AT32F405RCT7, U2 USBLC6-2SC6, U3 TLV75733PDBV, U4 XC6206P332MR, Y1 12MHz

Commit message: Replace the project with the reorganised T7 tree: ribbon keyboard is production, pogo archived
Production design is now the outward-facing FPC keyboard with per-key
SK6812MINI-E reverse-mount LEDs, a fifth SN74LV4051A mux per half so every
alternate Hall position has its own channel, an SN74AHCT1G125 LED level
shifter, a 50 x 31 mm daughterboard, 1.5 mm POM plates and 3 degree / 7 degree
tent and typing angles. The universal half panel is fully populated (359
placements) with routed NPTH alignment slots for the mutually exclusive
positions, and eight fixed-layout Left/Right PCB pairs are released under
release/layout-pcbs/ with matching BOM, CPL, Gerber ZIP, drill report and DRC.

Reorganise tools/ into cad/, generators/, layouts/, pcb/, pogo/, releases/ and
rendering/ subpackages; add designs/ and layout/ (KLE) trees and per-layout
gallery renders. The Fusion handoff is a fourteen-body reference STEP with
Gateron KS-20 switch and Cherry-profile keycap references and exact BOOMELE,
HRO and XKB models under case/fusion360/models/official/ with provenance.

The Neo-style pogo variant, its Mill-Max vendor models, the Fusion setup
script and the pogo release packages are archived as design history and
marked DO-NOT-ORDER. Their restored BOM snapshots had reintroduced the wrong
mux part C7792; corrected to C128414 / SN74LV4051ADR and their checksum lists
and archives rebuilt.

Co-Authored-By: Claude Opus 5 <noreply@anthropic.com>
Parts:
- added C16: 100n, symbol Symm60HE_Daughterboard_Symbols:SYM_C16
- added C17: 100n, symbol Symm60HE_Daughterboard_Symbols:SYM_C17
- added R5: 470R, symbol Symm60HE_Daughterboard_Symbols:SYM_R5
- added R6: 470R, symbol Symm60HE_Daughterboard_Symbols:SYM_R6
- added U5: SN74AHCT1G125, symbol Symm60HE_Daughterboard_Symbols:SYM_U5
- added U6: SN74AHCT1G125, symbol Symm60HE_Daughterboard_Symbols:SYM_U6
Connections:
- net +3V3A: now also J2.1 (+3V3A), J3.1 (+3V3A); no longer J2.12 (+3V3A), J3.12 (+3V3A)
- net ADC_L1: now also J2.7 (ADC_L1); no longer J2.6 (ADC_L1)
- net ADC_L2: now also J2.9 (ADC_L2); no longer J2.4 (ADC_L2)
- net ADC_L3: now also J2.11 (ADC_L3); no longer J2.2 (ADC_L3)
- net ADC_L4: now also J2.12 (ADC_L4); no longer J2.1 (ADC_L4)
- net ADC_R1: now also J3.7 (ADC_R1); no longer J3.6 (ADC_R1)
- net ADC_R2: now also J3.9 (ADC_R2); no longer J3.4 (ADC_R2)
- net ADC_R3: now also J3.11 (ADC_R3); no longer J3.2 (ADC_R3)
- net ADC_R4: now also J3.12 (ADC_R4); no longer J3.1 (ADC_R4)
- net GND: now also J2.8 (GND), J3.8 (GND), C16.2 (GND), C17.2 (GND), U5.1 (GND), U5.3 (GND), U6.1 (GND), U6.3 (GND); no longer J2.11 (GND), J2.3 (GND), J2.5 (GND), J2.7 (GND), J3.11 (GND), J3.3 (GND), J3.5 (GND), J3.7 (GND)
- net MUX_A0: now also J2.3 (MUX_A0), J3.3 (MUX_A0); no longer J2.10 (MUX_A0), J3.10 (MUX_A0)
- net MUX_A1: now also J2.4 (MUX_A1), J3.4 (MUX_A1); no longer J2.9 (MUX_A1), J3.9 (MUX_A1)
- net MUX_A2: now also J2.5 (MUX_A2), J3.5 (MUX_A2); no longer J2.8 (MUX_A2), J3.8 (MUX_A2)
- net VBUS: now also J2.6 (VBUS), J3.6 (VBUS), C16.1 (VBUS), C17.1 (VBUS), U5.5 (VBUS), U6.5 (VBUS)
- new net ADC_L5: J2.2 (ADC_L5), U1.16 (ADC_L5)
- new net ADC_R5: J3.2 (ADC_R5), U1.15 (ADC_R5)
- new net RGB_L: J2.10 (RGB_L), R5.2 (RGB_L)
- new net RGB_L_BUF: R5.1 (RGB_L_BUF), U5.4 (RGB_L_BUF)
- new net RGB_L_MCU: U1.8 (RGB_L_MCU), U5.2 (RGB_L_MCU)
- new net RGB_R: J3.10 (RGB_R), R6.2 (RGB_R)
- new net RGB_R_BUF: R6.1 (RGB_R_BUF), U6.4 (RGB_R_BUF)
- new net RGB_R_MCU: U1.41 (RGB_R_MCU), U6.2 (RGB_R_MCU)
