File: pcb/Symm60HE-Left.kicad_sch (KiCad schematic)
At the start: 109 parts

Commit message: Replace the project with the reorganised T7 tree: ribbon keyboard is production, pogo archived
Production design is now the outward-facing FPC keyboard with per-key
SK6812MINI-E reverse-mount LEDs, a fifth SN74LV4051A mux per half so every
alternate Hall position has its own channel, an SN74AHCT1G125 LED level
shifter, a 50 x 31 mm daughterboard, 1.5 mm POM plates and 3 degree / 7 degree
tent and typing angles. The universal half panel is fully populated (359
placements) with routed NPTH alignment slots for the mutually exclusive
positions, and eight fixed-layout Left/Right PCB pairs are released under
release/layout-pcbs/ with matching BOM, CPL, Gerber ZIP, drill report and DRC.

Reorganise tools/ into cad/, generators/, layouts/, pcb/, pogo/, releases/ and
rendering/ subpackages; add designs/ and layout/ (KLE) trees and per-layout
gallery renders. The Fusion handoff is a fourteen-body reference STEP with
Gateron KS-20 switch and Cherry-profile keycap references and exact BOOMELE,
HRO and XKB models under case/fusion360/models/official/ with provenance.

The Neo-style pogo variant, its Mill-Max vendor models, the Fusion setup
script and the pogo release packages are archived as design history and
marked DO-NOT-ORDER. Their restored BOM snapshots had reintroduced the wrong
mux part C7792; corrected to C128414 / SN74LV4051ADR and their checksum lists
and archives rebuilt.

Co-Authored-By: Claude Opus 5 <noreply@anthropic.com>
Parts:
- removed MHL1: M2, symbol Symm60HE_Left_Symbols:SYM_MHL1
- removed MHL2: M2, symbol Symm60HE_Left_Symbols:SYM_MHL2
- removed MHL3: M2, symbol Symm60HE_Left_Symbols:SYM_MHL3
- removed MHL4: M2, symbol Symm60HE_Left_Symbols:SYM_MHL4
- added AML5: SN74LV4051A, symbol Symm60HE_Left_Symbols:SYM_AML5
- added CL28A: 100n, symbol Symm60HE_Left_Symbols:SYM_CL28A
- added CL28B: 4.7n, symbol Symm60HE_Left_Symbols:SYM_CL28B
- added CML5: 100n, symbol Symm60HE_Left_Symbols:SYM_CML5
- added CRGBL1: 100n, symbol Symm60HE_Left_Symbols:SYM_CRGBL1
- added CRGBL10: 100n, symbol Symm60HE_Left_Symbols:SYM_CRGBL10
- added CRGBL11: 100n, symbol Symm60HE_Left_Symbols:SYM_CRGBL11
- added CRGBL12: 100n, symbol Symm60HE_Left_Symbols:SYM_CRGBL12
- added CRGBL13: 100n, symbol Symm60HE_Left_Symbols:SYM_CRGBL13
- added CRGBL14: 100n, symbol Symm60HE_Left_Symbols:SYM_CRGBL14
- added CRGBL15: 100n, symbol Symm60HE_Left_Symbols:SYM_CRGBL15
- added CRGBL16: 100n, symbol Symm60HE_Left_Symbols:SYM_CRGBL16
- added CRGBL17: 100n, symbol Symm60HE_Left_Symbols:SYM_CRGBL17
- added CRGBL18: 100n, symbol Symm60HE_Left_Symbols:SYM_CRGBL18
- added CRGBL19: 100n, symbol Symm60HE_Left_Symbols:SYM_CRGBL19
- added CRGBL2: 100n, symbol Symm60HE_Left_Symbols:SYM_CRGBL2
- added CRGBL20: 100n, symbol Symm60HE_Left_Symbols:SYM_CRGBL20
- added CRGBL21: 100n, symbol Symm60HE_Left_Symbols:SYM_CRGBL21
- added CRGBL22: 100n, symbol Symm60HE_Left_Symbols:SYM_CRGBL22
- added CRGBL23: 100n, symbol Symm60HE_Left_Symbols:SYM_CRGBL23
- added CRGBL24: 100n, symbol Symm60HE_Left_Symbols:SYM_CRGBL24
- added CRGBL25: 100n, symbol Symm60HE_Left_Symbols:SYM_CRGBL25
- added CRGBL26: 100n, symbol Symm60HE_Left_Symbols:SYM_CRGBL26
- added CRGBL27: 100n, symbol Symm60HE_Left_Symbols:SYM_CRGBL27
- added CRGBL29: 100n, symbol Symm60HE_Left_Symbols:SYM_CRGBL29
- added CRGBL3: 100n, symbol Symm60HE_Left_Symbols:SYM_CRGBL3
- added CRGBL30: 100n, symbol Symm60HE_Left_Symbols:SYM_CRGBL30
- added CRGBL31: 100n, symbol Symm60HE_Left_Symbols:SYM_CRGBL31
- added CRGBL33: 100n, symbol Symm60HE_Left_Symbols:SYM_CRGBL33
- added CRGBL4: 100n, symbol Symm60HE_Left_Symbols:SYM_CRGBL4
- added CRGBL5: 100n, symbol Symm60HE_Left_Symbols:SYM_CRGBL5
- added CRGBL6: 100n, symbol Symm60HE_Left_Symbols:SYM_CRGBL6
- added CRGBL7: 100n, symbol Symm60HE_Left_Symbols:SYM_CRGBL7
- added CRGBL8: 100n, symbol Symm60HE_Left_Symbols:SYM_CRGBL8
- added CRGBL9: 100n, symbol Symm60HE_Left_Symbols:SYM_CRGBL9
- added DL1: SK6812MINI-E, symbol Symm60HE_Left_Symbols:SYM_DL1
- added DL10: SK6812MINI-E, symbol Symm60HE_Left_Symbols:SYM_DL10
- added DL11: SK6812MINI-E, symbol Symm60HE_Left_Symbols:SYM_DL11
- added DL12: SK6812MINI-E, symbol Symm60HE_Left_Symbols:SYM_DL12
- added DL13: SK6812MINI-E, symbol Symm60HE_Left_Symbols:SYM_DL13
- added DL14: SK6812MINI-E, symbol Symm60HE_Left_Symbols:SYM_DL14
- added DL15: SK6812MINI-E, symbol Symm60HE_Left_Symbols:SYM_DL15
- added DL16: SK6812MINI-E, symbol Symm60HE_Left_Symbols:SYM_DL16
- added DL17: SK6812MINI-E, symbol Symm60HE_Left_Symbols:SYM_DL17
- added DL18: SK6812MINI-E, symbol Symm60HE_Left_Symbols:SYM_DL18
- added DL19: SK6812MINI-E, symbol Symm60HE_Left_Symbols:SYM_DL19
- added DL2: SK6812MINI-E, symbol Symm60HE_Left_Symbols:SYM_DL2
- added DL20: SK6812MINI-E, symbol Symm60HE_Left_Symbols:SYM_DL20
- added DL21: SK6812MINI-E, symbol Symm60HE_Left_Symbols:SYM_DL21
- added DL22: SK6812MINI-E, symbol Symm60HE_Left_Symbols:SYM_DL22
- added DL23: SK6812MINI-E, symbol Symm60HE_Left_Symbols:SYM_DL23
- added DL24: SK6812MINI-E, symbol Symm60HE_Left_Symbols:SYM_DL24
- added DL25: SK6812MINI-E, symbol Symm60HE_Left_Symbols:SYM_DL25
- added DL26: SK6812MINI-E, symbol Symm60HE_Left_Symbols:SYM_DL26
- added DL27: SK6812MINI-E, symbol Symm60HE_Left_Symbols:SYM_DL27
- added DL29: SK6812MINI-E, symbol Symm60HE_Left_Symbols:SYM_DL29
- added DL3: SK6812MINI-E, symbol Symm60HE_Left_Symbols:SYM_DL3
- added DL30: SK6812MINI-E, symbol Symm60HE_Left_Symbols:SYM_DL30
- added DL31: SK6812MINI-E, symbol Symm60HE_Left_Symbols:SYM_DL31
- added DL33: SK6812MINI-E, symbol Symm60HE_Left_Symbols:SYM_DL33
- added DL4: SK6812MINI-E, symbol Symm60HE_Left_Symbols:SYM_DL4
- added DL5: SK6812MINI-E, symbol Symm60HE_Left_Symbols:SYM_DL5
- added DL6: SK6812MINI-E, symbol Symm60HE_Left_Symbols:SYM_DL6
- added DL7: SK6812MINI-E, symbol Symm60HE_Left_Symbols:SYM_DL7
- added DL8: SK6812MINI-E, symbol Symm60HE_Left_Symbols:SYM_DL8
- added DL9: SK6812MINI-E, symbol Symm60HE_Left_Symbols:SYM_DL9
- added HEL28: MT9102ET, symbol Symm60HE_Left_Symbols:SYM_HEL28
- added RBPL29: 0R_DNP, symbol Symm60HE_Left_Symbols:SYM_RBPL29
Connections:
- net +3V3A: now also AML5.16 (+3V3A), CL28A.1 (+3V3A), CML5.1 (+3V3A), HEL28.1 (+3V3A)
- net GND: now also AML5.1 (GND), AML5.12 (GND), AML5.15 (GND), AML5.2 (GND), AML5.4 (GND), AML5.5 (GND), AML5.6 (GND), AML5.7 (GND), AML5.8 (GND), CL28A.2 (GND), CL28B.2 (GND), CML5.2 (GND), CRGBL1.2 (GND), CRGBL10.2 (GND), CRGBL11.2 (GND), CRGBL12.2 (GND), CRGBL13.2 (GND), CRGBL14.2 (GND), CRGBL15.2 (GND), CRGBL16.2 (GND), CRGBL17.2 (GND), CRGBL18.2 (GND), CRGBL19.2 (GND), CRGBL2.2 (GND), CRGBL20.2 (GND), CRGBL21.2 (GND), CRGBL22.2 (GND), CRGBL23.2 (GND), CRGBL24.2 (GND), CRGBL25.2 (GND), CRGBL26.2 (GND), CRGBL27.2 (GND), CRGBL29.2 (GND), CRGBL3.2 (GND), CRGBL30.2 (GND), CRGBL31.2 (GND), CRGBL33.2 (GND), CRGBL4.2 (GND), CRGBL5.2 (GND), CRGBL6.2 (GND), CRGBL7.2 (GND), CRGBL8.2 (GND), CRGBL9.2 (GND), DL1.1 (GND), DL10.1 (GND), DL11.1 (GND), DL12.1 (GND), DL13.1 (GND), DL14.1 (GND), DL15.1 (GND), DL16.1 (GND), DL17.1 (GND), DL18.1 (GND), DL19.1 (GND), DL2.1 (GND), DL20.1 (GND), DL21.1 (GND), DL22.1 (GND), DL23.1 (GND), DL24.1 (GND), DL25.1 (GND), DL26.1 (GND), DL27.1 (GND), DL29.1 (GND), DL3.1 (GND), DL30.1 (GND), DL31.1 (GND), DL33.1 (GND), DL4.1 (GND), DL5.1 (GND), DL6.1 (GND), DL7.1 (GND), DL8.1 (GND), DL9.1 (GND), HEL28.2 (GND); no longer JL1.11 (GND), JL1.3 (GND), JL1.7 (GND)
- net HE_L28: no longer CL30B.1 (HE_L28), HEL30.3 (HE_L28)
- net MUX_A0: now also AML5.11 (MUX_A0)
- net MUX_A1: now also AML5.10 (MUX_A1)
- net MUX_A2: now also AML5.9 (MUX_A2)
- new net ADC_L5: AML5.3 (ADC_L5), JL1.11 (ADC_L5)
- new net HE_L32: AML5.13 (HE_L32), CL28B.1 (HE_L32), HEL28.3 (HE_L32)
- new net HE_L33: AML5.14 (HE_L33), CL30B.1 (HE_L33), HEL30.3 (HE_L33)
- new net RGB_L: DL1.2 (RGB_L), JL1.3 (RGB_L)
- new net RGB_L_01: DL1.4 (RGB_L_01), DL2.2 (RGB_L_01)
- new net RGB_L_02: DL2.4 (RGB_L_02), DL3.2 (RGB_L_02)
- new net RGB_L_03: DL3.4 (RGB_L_03), DL4.2 (RGB_L_03)
- new net RGB_L_04: DL4.4 (RGB_L_04), DL5.2 (RGB_L_04)
- new net RGB_L_05: DL5.4 (RGB_L_05), DL6.2 (RGB_L_05)
- new net RGB_L_06: DL6.4 (RGB_L_06), DL7.2 (RGB_L_06)
- new net RGB_L_07: DL7.4 (RGB_L_07), DL8.2 (RGB_L_07)
- new net RGB_L_08: DL8.4 (RGB_L_08), DL9.2 (RGB_L_08)
- new net RGB_L_09: DL10.2 (RGB_L_09), DL9.4 (RGB_L_09)
- new net RGB_L_10: DL10.4 (RGB_L_10), DL11.2 (RGB_L_10)
- new net RGB_L_11: DL11.4 (RGB_L_11), DL12.2 (RGB_L_11)
- new net RGB_L_12: DL12.4 (RGB_L_12), DL13.2 (RGB_L_12)
- new net RGB_L_13: DL13.4 (RGB_L_13), DL14.2 (RGB_L_13)
- new net RGB_L_14: DL14.4 (RGB_L_14), DL15.2 (RGB_L_14)
- new net RGB_L_15: DL15.4 (RGB_L_15), DL16.2 (RGB_L_15)
- new net RGB_L_16: DL16.4 (RGB_L_16), DL17.2 (RGB_L_16)
- new net RGB_L_17: DL17.4 (RGB_L_17), DL18.2 (RGB_L_17)
- new net RGB_L_18: DL18.4 (RGB_L_18), DL19.2 (RGB_L_18)
- new net RGB_L_19: DL19.4 (RGB_L_19), DL20.2 (RGB_L_19)
- new net RGB_L_20: DL20.4 (RGB_L_20), DL21.2 (RGB_L_20)
- new net RGB_L_21: DL21.4 (RGB_L_21), DL22.2 (RGB_L_21)
- new net RGB_L_22: DL22.4 (RGB_L_22), DL23.2 (RGB_L_22)
- new net RGB_L_23: DL23.4 (RGB_L_23), DL24.2 (RGB_L_23)
- new net RGB_L_24: DL24.4 (RGB_L_24), DL25.2 (RGB_L_24)
- new net RGB_L_25: DL25.4 (RGB_L_25), DL26.2 (RGB_L_25)
- new net RGB_L_26: DL26.4 (RGB_L_26), DL27.2 (RGB_L_26)
- new net RGB_L_27: DL27.4 (RGB_L_27), DL33.2 (RGB_L_27)
- new net RGB_L_28: DL29.2 (RGB_L_28), DL33.4 (RGB_L_28), RBPL29.1 (RGB_L_28)
- new net RGB_L_29: DL29.4 (RGB_L_29), DL30.2 (RGB_L_29), RBPL29.2 (RGB_L_29)
- new net RGB_L_30: DL30.4 (RGB_L_30), DL31.2 (RGB_L_30)
- new net VBUS: CRGBL1.1 (VBUS), CRGBL10.1 (VBUS), CRGBL11.1 (VBUS), CRGBL12.1 (VBUS), CRGBL13.1 (VBUS), CRGBL14.1 (VBUS), CRGBL15.1 (VBUS), CRGBL16.1 (VBUS), CRGBL17.1 (VBUS), CRGBL18.1 (VBUS), CRGBL19.1 (VBUS), CRGBL2.1 (VBUS), CRGBL20.1 (VBUS), CRGBL21.1 (VBUS), CRGBL22.1 (VBUS), CRGBL23.1 (VBUS), CRGBL24.1 (VBUS), CRGBL25.1 (VBUS), CRGBL26.1 (VBUS), CRGBL27.1 (VBUS), CRGBL29.1 (VBUS), CRGBL3.1 (VBUS), CRGBL30.1 (VBUS), CRGBL31.1 (VBUS), CRGBL33.1 (VBUS), CRGBL4.1 (VBUS), CRGBL5.1 (VBUS), CRGBL6.1 (VBUS), CRGBL7.1 (VBUS), CRGBL8.1 (VBUS), CRGBL9.1 (VBUS), DL1.3 (VBUS), DL10.3 (VBUS), DL11.3 (VBUS), DL12.3 (VBUS), DL13.3 (VBUS), DL14.3 (VBUS), DL15.3 (VBUS), DL16.3 (VBUS), DL17.3 (VBUS), DL18.3 (VBUS), DL19.3 (VBUS), DL2.3 (VBUS), DL20.3 (VBUS), DL21.3 (VBUS), DL22.3 (VBUS), DL23.3 (VBUS), DL24.3 (VBUS), DL25.3 (VBUS), DL26.3 (VBUS), DL27.3 (VBUS), DL29.3 (VBUS), DL3.3 (VBUS), DL30.3 (VBUS), DL31.3 (VBUS), DL33.3 (VBUS), DL4.3 (VBUS), DL5.3 (VBUS), DL6.3 (VBUS), DL7.3 (VBUS), DL8.3 (VBUS), DL9.3 (VBUS), JL1.7 (VBUS)
- no-connect marks 0 -> 1
