File: pcb/Symm60HE-Right.kicad_sch (KiCad schematic)
At the start: 118 parts

Commit message: Replace the project with the reorganised T7 tree: ribbon keyboard is production, pogo archived
Production design is now the outward-facing FPC keyboard with per-key
SK6812MINI-E reverse-mount LEDs, a fifth SN74LV4051A mux per half so every
alternate Hall position has its own channel, an SN74AHCT1G125 LED level
shifter, a 50 x 31 mm daughterboard, 1.5 mm POM plates and 3 degree / 7 degree
tent and typing angles. The universal half panel is fully populated (359
placements) with routed NPTH alignment slots for the mutually exclusive
positions, and eight fixed-layout Left/Right PCB pairs are released under
release/layout-pcbs/ with matching BOM, CPL, Gerber ZIP, drill report and DRC.

Reorganise tools/ into cad/, generators/, layouts/, pcb/, pogo/, releases/ and
rendering/ subpackages; add designs/ and layout/ (KLE) trees and per-layout
gallery renders. The Fusion handoff is a fourteen-body reference STEP with
Gateron KS-20 switch and Cherry-profile keycap references and exact BOOMELE,
HRO and XKB models under case/fusion360/models/official/ with provenance.

The Neo-style pogo variant, its Mill-Max vendor models, the Fusion setup
script and the pogo release packages are archived as design history and
marked DO-NOT-ORDER. Their restored BOM snapshots had reintroduced the wrong
mux part C7792; corrected to C128414 / SN74LV4051ADR and their checksum lists
and archives rebuilt.

Co-Authored-By: Claude Opus 5 <noreply@anthropic.com>
Parts:
- removed MHR1: M2, symbol Symm60HE_Right_Symbols:SYM_MHR1
- removed MHR2: M2, symbol Symm60HE_Right_Symbols:SYM_MHR2
- removed MHR3: M2, symbol Symm60HE_Right_Symbols:SYM_MHR3
- removed MHR4: M2, symbol Symm60HE_Right_Symbols:SYM_MHR4
- added AMR5: SN74LV4051A, symbol Symm60HE_Right_Symbols:SYM_AMR5
- added CMR5: 100n, symbol Symm60HE_Right_Symbols:SYM_CMR5
- added CR31A: 100n, symbol Symm60HE_Right_Symbols:SYM_CR31A
- added CR31B: 4.7n, symbol Symm60HE_Right_Symbols:SYM_CR31B
- added CRGBR1: 100n, symbol Symm60HE_Right_Symbols:SYM_CRGBR1
- added CRGBR10: 100n, symbol Symm60HE_Right_Symbols:SYM_CRGBR10
- added CRGBR11: 100n, symbol Symm60HE_Right_Symbols:SYM_CRGBR11
- added CRGBR12: 100n, symbol Symm60HE_Right_Symbols:SYM_CRGBR12
- added CRGBR13: 100n, symbol Symm60HE_Right_Symbols:SYM_CRGBR13
- added CRGBR14: 100n, symbol Symm60HE_Right_Symbols:SYM_CRGBR14
- added CRGBR15: 100n, symbol Symm60HE_Right_Symbols:SYM_CRGBR15
- added CRGBR16: 100n, symbol Symm60HE_Right_Symbols:SYM_CRGBR16
- added CRGBR17: 100n, symbol Symm60HE_Right_Symbols:SYM_CRGBR17
- added CRGBR18: 100n, symbol Symm60HE_Right_Symbols:SYM_CRGBR18
- added CRGBR19: 100n, symbol Symm60HE_Right_Symbols:SYM_CRGBR19
- added CRGBR2: 100n, symbol Symm60HE_Right_Symbols:SYM_CRGBR2
- added CRGBR20: 100n, symbol Symm60HE_Right_Symbols:SYM_CRGBR20
- added CRGBR21: 100n, symbol Symm60HE_Right_Symbols:SYM_CRGBR21
- added CRGBR22: 100n, symbol Symm60HE_Right_Symbols:SYM_CRGBR22
- added CRGBR23: 100n, symbol Symm60HE_Right_Symbols:SYM_CRGBR23
- added CRGBR24: 100n, symbol Symm60HE_Right_Symbols:SYM_CRGBR24
- added CRGBR25: 100n, symbol Symm60HE_Right_Symbols:SYM_CRGBR25
- added CRGBR26: 100n, symbol Symm60HE_Right_Symbols:SYM_CRGBR26
- added CRGBR27: 100n, symbol Symm60HE_Right_Symbols:SYM_CRGBR27
- added CRGBR28: 100n, symbol Symm60HE_Right_Symbols:SYM_CRGBR28
- added CRGBR29: 100n, symbol Symm60HE_Right_Symbols:SYM_CRGBR29
- added CRGBR3: 100n, symbol Symm60HE_Right_Symbols:SYM_CRGBR3
- added CRGBR31: 100n, symbol Symm60HE_Right_Symbols:SYM_CRGBR31
- added CRGBR32: 100n, symbol Symm60HE_Right_Symbols:SYM_CRGBR32
- added CRGBR33: 100n, symbol Symm60HE_Right_Symbols:SYM_CRGBR33
- added CRGBR34: 100n, symbol Symm60HE_Right_Symbols:SYM_CRGBR34
- added CRGBR36: 100n, symbol Symm60HE_Right_Symbols:SYM_CRGBR36
- added CRGBR4: 100n, symbol Symm60HE_Right_Symbols:SYM_CRGBR4
- added CRGBR5: 100n, symbol Symm60HE_Right_Symbols:SYM_CRGBR5
- added CRGBR6: 100n, symbol Symm60HE_Right_Symbols:SYM_CRGBR6
- added CRGBR7: 100n, symbol Symm60HE_Right_Symbols:SYM_CRGBR7
- added CRGBR8: 100n, symbol Symm60HE_Right_Symbols:SYM_CRGBR8
- added CRGBR9: 100n, symbol Symm60HE_Right_Symbols:SYM_CRGBR9
- added DR1: SK6812MINI-E, symbol Symm60HE_Right_Symbols:SYM_DR1
- added DR10: SK6812MINI-E, symbol Symm60HE_Right_Symbols:SYM_DR10
- added DR11: SK6812MINI-E, symbol Symm60HE_Right_Symbols:SYM_DR11
- added DR12: SK6812MINI-E, symbol Symm60HE_Right_Symbols:SYM_DR12
- added DR13: SK6812MINI-E, symbol Symm60HE_Right_Symbols:SYM_DR13
- added DR14: SK6812MINI-E, symbol Symm60HE_Right_Symbols:SYM_DR14
- added DR15: SK6812MINI-E, symbol Symm60HE_Right_Symbols:SYM_DR15
- added DR16: SK6812MINI-E, symbol Symm60HE_Right_Symbols:SYM_DR16
- added DR17: SK6812MINI-E, symbol Symm60HE_Right_Symbols:SYM_DR17
- added DR18: SK6812MINI-E, symbol Symm60HE_Right_Symbols:SYM_DR18
- added DR19: SK6812MINI-E, symbol Symm60HE_Right_Symbols:SYM_DR19
- added DR2: SK6812MINI-E, symbol Symm60HE_Right_Symbols:SYM_DR2
- added DR20: SK6812MINI-E, symbol Symm60HE_Right_Symbols:SYM_DR20
- added DR21: SK6812MINI-E, symbol Symm60HE_Right_Symbols:SYM_DR21
- added DR22: SK6812MINI-E, symbol Symm60HE_Right_Symbols:SYM_DR22
- added DR23: SK6812MINI-E, symbol Symm60HE_Right_Symbols:SYM_DR23
- added DR24: SK6812MINI-E, symbol Symm60HE_Right_Symbols:SYM_DR24
- added DR25: SK6812MINI-E, symbol Symm60HE_Right_Symbols:SYM_DR25
- added DR26: SK6812MINI-E, symbol Symm60HE_Right_Symbols:SYM_DR26
- added DR27: SK6812MINI-E, symbol Symm60HE_Right_Symbols:SYM_DR27
- added DR28: SK6812MINI-E, symbol Symm60HE_Right_Symbols:SYM_DR28
- added DR29: SK6812MINI-E, symbol Symm60HE_Right_Symbols:SYM_DR29
- added DR3: SK6812MINI-E, symbol Symm60HE_Right_Symbols:SYM_DR3
- added DR31: SK6812MINI-E, symbol Symm60HE_Right_Symbols:SYM_DR31
- added DR32: SK6812MINI-E, symbol Symm60HE_Right_Symbols:SYM_DR32
- added DR33: SK6812MINI-E, symbol Symm60HE_Right_Symbols:SYM_DR33
- added DR34: SK6812MINI-E, symbol Symm60HE_Right_Symbols:SYM_DR34
- added DR36: SK6812MINI-E, symbol Symm60HE_Right_Symbols:SYM_DR36
- added DR4: SK6812MINI-E, symbol Symm60HE_Right_Symbols:SYM_DR4
- added DR5: SK6812MINI-E, symbol Symm60HE_Right_Symbols:SYM_DR5
- added DR6: SK6812MINI-E, symbol Symm60HE_Right_Symbols:SYM_DR6
- added DR7: SK6812MINI-E, symbol Symm60HE_Right_Symbols:SYM_DR7
- added DR8: SK6812MINI-E, symbol Symm60HE_Right_Symbols:SYM_DR8
- added DR9: SK6812MINI-E, symbol Symm60HE_Right_Symbols:SYM_DR9
- added HER31: MT9102ET, symbol Symm60HE_Right_Symbols:SYM_HER31
- added RBPR24: 0R_DNP, symbol Symm60HE_Right_Symbols:SYM_RBPR24
- added RBPR31: 0R_DNP, symbol Symm60HE_Right_Symbols:SYM_RBPR31
- added RBPR5: 0R_DNP, symbol Symm60HE_Right_Symbols:SYM_RBPR5
Connections:
- net +3V3A: now also AMR5.16 (+3V3A), CMR5.1 (+3V3A), CR31A.1 (+3V3A), HER31.1 (+3V3A)
- net GND: now also AMR5.1 (GND), AMR5.2 (GND), AMR5.4 (GND), AMR5.5 (GND), AMR5.6 (GND), AMR5.7 (GND), AMR5.8 (GND), CMR5.2 (GND), CR31A.2 (GND), CR31B.2 (GND), CRGBR1.2 (GND), CRGBR10.2 (GND), CRGBR11.2 (GND), CRGBR12.2 (GND), CRGBR13.2 (GND), CRGBR14.2 (GND), CRGBR15.2 (GND), CRGBR16.2 (GND), CRGBR17.2 (GND), CRGBR18.2 (GND), CRGBR19.2 (GND), CRGBR2.2 (GND), CRGBR20.2 (GND), CRGBR21.2 (GND), CRGBR22.2 (GND), CRGBR23.2 (GND), CRGBR24.2 (GND), CRGBR25.2 (GND), CRGBR26.2 (GND), CRGBR27.2 (GND), CRGBR28.2 (GND), CRGBR29.2 (GND), CRGBR3.2 (GND), CRGBR31.2 (GND), CRGBR32.2 (GND), CRGBR33.2 (GND), CRGBR34.2 (GND), CRGBR36.2 (GND), CRGBR4.2 (GND), CRGBR5.2 (GND), CRGBR6.2 (GND), CRGBR7.2 (GND), CRGBR8.2 (GND), CRGBR9.2 (GND), DR1.1 (GND), DR10.1 (GND), DR11.1 (GND), DR12.1 (GND), DR13.1 (GND), DR14.1 (GND), DR15.1 (GND), DR16.1 (GND), DR17.1 (GND), DR18.1 (GND), DR19.1 (GND), DR2.1 (GND), DR20.1 (GND), DR21.1 (GND), DR22.1 (GND), DR23.1 (GND), DR24.1 (GND), DR25.1 (GND), DR26.1 (GND), DR27.1 (GND), DR28.1 (GND), DR29.1 (GND), DR3.1 (GND), DR31.1 (GND), DR32.1 (GND), DR33.1 (GND), DR34.1 (GND), DR36.1 (GND), DR4.1 (GND), DR5.1 (GND), DR6.1 (GND), DR7.1 (GND), DR8.1 (GND), DR9.1 (GND), HER31.2 (GND); no longer JR1.10 (GND), JR1.2 (GND), JR1.6 (GND)
- net HE_R04: no longer CR4B.1 (HE_R04), HER4.3 (HE_R04)
- net HE_R25: no longer CR26B.1 (HE_R25), HER26.3 (HE_R25)
- net HE_R30: no longer CR33B.1 (HE_R30), HER33.3 (HE_R30)
- net MUX_A0: now also AMR5.11 (MUX_A0)
- net MUX_A1: now also AMR5.10 (MUX_A1)
- net MUX_A2: now also AMR5.9 (MUX_A2)
- new net ADC_R5: AMR5.3 (ADC_R5), JR1.2 (ADC_R5)
- new net HE_R33: AMR5.13 (HE_R33), CR4B.1 (HE_R33), HER4.3 (HE_R33)
- new net HE_R34: AMR5.14 (HE_R34), CR26B.1 (HE_R34), HER26.3 (HE_R34)
- new net HE_R35: AMR5.15 (HE_R35), CR31B.1 (HE_R35), HER31.3 (HE_R35)
- new net HE_R36: AMR5.12 (HE_R36), CR33B.1 (HE_R36), HER33.3 (HE_R36)
- new net RGB_R: DR1.2 (RGB_R), JR1.10 (RGB_R)
- new net RGB_R_01: DR1.4 (RGB_R_01), DR2.2 (RGB_R_01)
- new net RGB_R_02: DR2.4 (RGB_R_02), DR3.2 (RGB_R_02)
- new net RGB_R_03: DR3.4 (RGB_R_03), DR33.2 (RGB_R_03), DR4.2 (RGB_R_03)
- new net RGB_R_04: DR33.4 (RGB_R_04), DR4.4 (RGB_R_04), DR5.2 (RGB_R_04), RBPR5.1 (RGB_R_04)
- new net RGB_R_05: DR5.4 (RGB_R_05), DR6.2 (RGB_R_05), RBPR5.2 (RGB_R_05)
- new net RGB_R_06: DR6.4 (RGB_R_06), DR7.2 (RGB_R_06)
- new net RGB_R_07: DR7.4 (RGB_R_07), DR8.2 (RGB_R_07)
- new net RGB_R_08: DR8.4 (RGB_R_08), DR9.2 (RGB_R_08)
- new net RGB_R_09: DR10.2 (RGB_R_09), DR9.4 (RGB_R_09)
- new net RGB_R_10: DR10.4 (RGB_R_10), DR11.2 (RGB_R_10)
- new net RGB_R_11: DR11.4 (RGB_R_11), DR12.2 (RGB_R_11)
- new net RGB_R_12: DR12.4 (RGB_R_12), DR13.2 (RGB_R_12)
- new net RGB_R_13: DR13.4 (RGB_R_13), DR14.2 (RGB_R_13)
- new net RGB_R_14: DR14.4 (RGB_R_14), DR15.2 (RGB_R_14)
- new net RGB_R_15: DR15.4 (RGB_R_15), DR16.2 (RGB_R_15)
- new net RGB_R_16: DR16.4 (RGB_R_16), DR17.2 (RGB_R_16)
- new net RGB_R_17: DR17.4 (RGB_R_17), DR18.2 (RGB_R_17)
- new net RGB_R_18: DR18.4 (RGB_R_18), DR19.2 (RGB_R_18)
- new net RGB_R_19: DR19.4 (RGB_R_19), DR20.2 (RGB_R_19)
- new net RGB_R_20: DR20.4 (RGB_R_20), DR21.2 (RGB_R_20), DR34.2 (RGB_R_20)
- new net RGB_R_21: DR21.4 (RGB_R_21), DR22.2 (RGB_R_21), DR34.4 (RGB_R_21)
- new net RGB_R_22: DR22.4 (RGB_R_22), DR23.2 (RGB_R_22)
- new net RGB_R_23: DR23.4 (RGB_R_23), DR24.2 (RGB_R_23), RBPR24.1 (RGB_R_23)
- new net RGB_R_24: DR24.4 (RGB_R_24), DR25.2 (RGB_R_24), RBPR24.2 (RGB_R_24)
- new net RGB_R_25: DR25.4 (RGB_R_25), DR26.2 (RGB_R_25)
- new net RGB_R_26: DR26.4 (RGB_R_26), DR27.2 (RGB_R_26)
- new net RGB_R_27: DR27.4 (RGB_R_27), DR28.2 (RGB_R_27)
- new net RGB_R_28: DR28.4 (RGB_R_28), DR29.2 (RGB_R_28)
- new net RGB_R_29: DR29.4 (RGB_R_29), DR36.2 (RGB_R_29)
- new net RGB_R_30: DR31.2 (RGB_R_30), DR36.4 (RGB_R_30), RBPR31.1 (RGB_R_30)
- new net RGB_R_31: DR31.4 (RGB_R_31), DR32.2 (RGB_R_31), RBPR31.2 (RGB_R_31)
- new net VBUS: CRGBR1.1 (VBUS), CRGBR10.1 (VBUS), CRGBR11.1 (VBUS), CRGBR12.1 (VBUS), CRGBR13.1 (VBUS), CRGBR14.1 (VBUS), CRGBR15.1 (VBUS), CRGBR16.1 (VBUS), CRGBR17.1 (VBUS), CRGBR18.1 (VBUS), CRGBR19.1 (VBUS), CRGBR2.1 (VBUS), CRGBR20.1 (VBUS), CRGBR21.1 (VBUS), CRGBR22.1 (VBUS), CRGBR23.1 (VBUS), CRGBR24.1 (VBUS), CRGBR25.1 (VBUS), CRGBR26.1 (VBUS), CRGBR27.1 (VBUS), CRGBR28.1 (VBUS), CRGBR29.1 (VBUS), CRGBR3.1 (VBUS), CRGBR31.1 (VBUS), CRGBR32.1 (VBUS), CRGBR33.1 (VBUS), CRGBR34.1 (VBUS), CRGBR36.1 (VBUS), CRGBR4.1 (VBUS), CRGBR5.1 (VBUS), CRGBR6.1 (VBUS), CRGBR7.1 (VBUS), CRGBR8.1 (VBUS), CRGBR9.1 (VBUS), DR1.3 (VBUS), DR10.3 (VBUS), DR11.3 (VBUS), DR12.3 (VBUS), DR13.3 (VBUS), DR14.3 (VBUS), DR15.3 (VBUS), DR16.3 (VBUS), DR17.3 (VBUS), DR18.3 (VBUS), DR19.3 (VBUS), DR2.3 (VBUS), DR20.3 (VBUS), DR21.3 (VBUS), DR22.3 (VBUS), DR23.3 (VBUS), DR24.3 (VBUS), DR25.3 (VBUS), DR26.3 (VBUS), DR27.3 (VBUS), DR28.3 (VBUS), DR29.3 (VBUS), DR3.3 (VBUS), DR31.3 (VBUS), DR32.3 (VBUS), DR33.3 (VBUS), DR34.3 (VBUS), DR36.3 (VBUS), DR4.3 (VBUS), DR5.3 (VBUS), DR6.3 (VBUS), DR7.3 (VBUS), DR8.3 (VBUS), DR9.3 (VBUS), JR1.6 (VBUS)
- no-connect marks 0 -> 1
