File: pcb/Symm60HE-Panel-SideBySide.kicad_pcb (KiCad board)
At the start: 2 copper layers, 162.3 x 227.8 mm, 448 parts

Commit message: Add a side-by-side panel, refresh the Fusion handoff
Both panel arrangements are now generated. The stacked one stays the panel the
release orders, because it is the cheaper of the two in both the ways that
matter for board price: 369.7 against 375.7 cm2 of material, and a 227.8 mm
longest edge against 310.2 mm. The side-by-side arrangement keeps the halves in
the orientation they are assembled in, joined across the centre gap by two
tabs, with three tabs per board on the top and bottom rails and one on each
outer rail; two of its tabs slide along the rail to keep their mouse bites off
board copper, the same way the stacked panel's do.

The Fusion reference solids were still the ones exported before the LEDs moved.
Regenerating them on Windows turned up three things the preparation script only
knew how to do on a Mac: it looked for KiCad's Python and 3D model library
under /opt/homebrew, and when given Windows paths as well it sorted them as
text, so "9.0" beat "10.0" -- and KiCad 9's library has no reverse-mount
SK6812MINI-E, so all 65 LEDs dropped silently out of the component export. Both
searches now compare version numbers, SYMM60_KICAD_PYTHON overrides the first,
and a machine without OpenSCAD gets the board solids with a note about the
plates rather than an error and nothing. build.sh finds FreeCAD the same way,
including FreeCADCmd.exe on Windows.

The Fusion setup script was still the pogo-era one: it pointed at a drive that
no longer holds the repository and imported target connectors, spring PCBs and
travel envelopes that this design does not have. It now imports the fourteen
parts the tree actually exports, keeps the ribbon routes hidden in their own
group, and checks that nothing arrived empty -- which is the failure worth
catching, unlike the placement manifest it used to verify against, which no
longer describes assembled positions. It lives in the repository now, beside
the references it reads.

Co-Authored-By: Claude Opus 5 <noreply@anthropic.com>
Parts:
- added MB66: MOUSE_BITE_0.5MM, MouseBite_0.5mm, F.Cu at (146.4, 72.1)
- added MB67: MOUSE_BITE_0.5MM, MouseBite_0.5mm, F.Cu at (146.4, 72.9)
- added MB68: MOUSE_BITE_0.5MM, MouseBite_0.5mm, F.Cu at (146.4, 73.6)
- added MB69: MOUSE_BITE_0.5MM, MouseBite_0.5mm, F.Cu at (146.4, 74.4)
- added MB70: MOUSE_BITE_0.5MM, MouseBite_0.5mm, F.Cu at (146.4, 75.1)
- added MB71: MOUSE_BITE_0.5MM, MouseBite_0.5mm, F.Cu at (-0.45, 51.2)
- added MB72: MOUSE_BITE_0.5MM, MouseBite_0.5mm, F.Cu at (-0.45, 51.9)
- added MB73: MOUSE_BITE_0.5MM, MouseBite_0.5mm, F.Cu at (-0.45, 52.7)
- added MB74: MOUSE_BITE_0.5MM, MouseBite_0.5mm, F.Cu at (-0.45, 53.4)
- added MB75: MOUSE_BITE_0.5MM, MouseBite_0.5mm, F.Cu at (-0.45, 54.2)
- added MB76: MOUSE_BITE_0.5MM, MouseBite_0.5mm, F.Cu at (293.3, 51.2)
- added MB77: MOUSE_BITE_0.5MM, MouseBite_0.5mm, F.Cu at (293.3, 51.9)
- added MB78: MOUSE_BITE_0.5MM, MouseBite_0.5mm, F.Cu at (293.3, 52.7)
- added MB79: MOUSE_BITE_0.5MM, MouseBite_0.5mm, F.Cu at (293.3, 53.4)
- added MB80: MOUSE_BITE_0.5MM, MouseBite_0.5mm, F.Cu at (293.3, 54.2)
- moved MB60 262.8 mm to (255.3, 94.8)
- moved MB59 261.8 mm to (254.5, 94.8)
- moved MB58 260.9 mm to (253.8, 94.8)
- moved MB57 260.0 mm to (253.0, 94.8)
- moved MB56 259.1 mm to (252.3, 94.8)
- moved MB41 231.0 mm to (218.9, 0.81)
- moved MB42 231.0 mm to (219.6, 0.81)
- moved MB43 231.0 mm to (220.4, 0.81)
- moved MB44 231.0 mm to (221.1, 0.81)
- moved MB45 231.0 mm to (221.9, 0.81)
- moved MB50 226.0 mm to (221.9, 94.8)
- moved MB49 225.4 mm to (221.1, 94.8)
- moved MB48 224.8 mm to (220.4, 94.8)
- moved MB47 224.2 mm to (219.6, 94.8)
- moved MB46 223.6 mm to (218.9, 94.8)
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Other:
- board size 162.3 x 227.8 mm -> 310.2 x 121.1 mm
