File: pcb/Symm60HE-Daughterboard.kicad_pcb (KiCad board)
At the start: 2 copper layers, 50 x 31 mm, 40 parts, among them J1 TYPE-C-31-M-12, J2 FFC_12P, J3 FFC_12P, SW1 TS-1187A, SW2 TS-1187A, U1 AT32F405RCT7, U2 USBLC6-2SC6, U3 TLV75733PDBV, U4 XC6206P332MR, U5 SN74AHCT1G125, U6 SN74AHCT1G125, Y1 12MHz

Commit message: Publish 2026-10-05 production PCBs and firmware
Routing:
- net GND: track 240.7 -> 0.00 mm, vias 6 -> 5
- net VBUS: track 114.8 -> 111.2 mm
Other:
- board size 50 x 31 mm -> 49.5 x 29.2 mm
