File: pcb/Symm60HE-Left.kicad_pcb (KiCad board)
At the start: 2 copper layers, 145.9 x 104.7 mm, 179 parts

Commit message: Publish 2026-10-05 production PCBs and firmware
Parts:
- AML1, AML2, AML3, AML4, AML5: footprint Symm60HE_Project:AM1_SOIC-16_3.9x9.9mm_P1.27mm -> Symm60HE_Project:AM1_TSSOP-16_4.4x5mm_P0.65mm
- moved AML2 0.93 mm to (33.8, 40.0)
Routing:
- net HE_L02: track 41.2 -> 112.0 mm, vias 0 -> 10
- net HE_L07: track 137.5 -> 179.2 mm, vias 2 -> 10
- net MUX_A0: track 244.1 -> 268.8 mm, vias 4 -> 15
- net HE_L03: track 54.0 -> 78.0 mm, vias 0 -> 8
- net MUX_A1: track 260.8 -> 280.0 mm, vias 3 -> 4
- net +3V3A: track 1059.3 -> 1069.5 mm
- net MUX_A2: track 224.2 -> 234.3 mm, vias 4 -> 9
- net RGB_L_27: track 25.3 -> 16.2 mm, vias 2 -> 0
- net HE_L04: track 76.3 -> 84.4 mm, vias 2 -> 6
- net RGB_L_26: track 133.9 -> 127.8 mm, vias 3 -> 2
- net HE_L23: track 14.0 -> 19.7 mm
- net HE_L19: track 47.7 -> 52.7 mm
- net HE_L29: track 30.9 -> 35.9 mm
- net HE_L12: track 89.0 -> 93.8 mm
- net GND: track 47.2 -> 51.9 mm
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