File: pcb/Symm60HE-Panel.kicad_pcb (KiCad board)
At the start: 2 copper layers, 162.3 x 227.8 mm, 448 parts

Commit message: Publish 2026-10-05 production PCBs and firmware
Parts:
- L-AML1, L-AML2, L-AML3, L-AML4, L-AML5, R-AMR1, R-AMR2, R-AMR3, R-AMR4, R-AMR5: footprint Symm60HE_Project:AM1_SOIC-16_3.9x9.9mm_P1.27mm -> Symm60HE_Project:AM1_TSSOP-16_4.4x5mm_P0.65mm
- moved MB41 1.51 mm to (105.9, 201.6)
- moved MB42 1.51 mm to (106.6, 201.6)
- moved MB43 1.51 mm to (107.4, 201.6)
- moved MB44 1.51 mm to (108.1, 201.6)
- moved MB45 1.51 mm to (108.9, 201.6)
- moved MB36 1.50 mm to (105.9, 103.7)
- moved MB37 1.50 mm to (106.6, 103.7)
- moved MB38 1.50 mm to (107.4, 103.7)
- moved MB39 1.50 mm to (108.1, 103.7)
- moved MB40 1.50 mm to (108.9, 103.7)
- moved MB31 1.50 mm to (105.9, 4.35)
- moved MB32 1.50 mm to (106.6, 4.35)
- moved MB33 1.50 mm to (107.4, 4.35)
- moved MB34 1.50 mm to (108.1, 4.35)
- moved MB35 1.50 mm to (108.9, 4.35)
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Connections:
- R-AMR1 pad 4: /R/HE_R08 -> /R/GND
- R-AMR1 pad 8: /R/GND -> /R/HE_R08
Routing:
- net /L/HE_L02: track 41.2 -> 112.0 mm, vias 0 -> 10
- net /R/HE_R07: track 127.4 -> 182.7 mm, vias 2 -> 6
- net /R/HE_R05: track 54.1 -> 103.0 mm, vias 2 -> 10
- net /L/HE_L07: track 137.5 -> 182.7 mm, vias 2 -> 10
- net /R/MUX_A0: track 254.2 -> 298.0 mm, vias 9 -> 11
- net /R/RGB_R_21: track 100.5 -> 58.2 mm, vias 6 -> 4
- net /R/RGB_R_17: track 55.1 -> 21.5 mm, vias 4 -> 2
- net /L/HE_L03: track 54.0 -> 79.9 mm, vias 0 -> 8
- net /L/MUX_A0: track 244.1 -> 268.8 mm, vias 4 -> 15
- net /R/+3V3A: track 1042.2 -> 1065.7 mm, vias 27 -> 37
- net /R/MUX_A2: track 184.2 -> 206.8 mm, vias 7 -> 13
- net /R/HE_R20: track 72.4 -> 94.3 mm, vias 2 -> 10
- net /L/MUX_A1: track 260.8 -> 280.0 mm, vias 3 -> 4
- net /L/+3V3A: track 1059.3 -> 1077.7 mm
- net /R/HE_R08: track 93.9 -> 111.7 mm, vias 2 -> 6
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Other:
- outline, holes or cut-outs redrawn
