File: pcb/Symm60HE-Right.kicad_pcb (KiCad board)
At the start: 2 copper layers, 145.9 x 104.7 mm, 197 parts

Commit message: Publish 2026-10-05 production PCBs and firmware
Parts:
- AMR1, AMR2, AMR3, AMR4, AMR5: footprint Symm60HE_Project:AM1_SOIC-16_3.9x9.9mm_P1.27mm -> Symm60HE_Project:AM1_TSSOP-16_4.4x5mm_P0.65mm
- moved AMR2 0.93 mm to (268.6, 40.0)
Connections:
- AMR1 pad 4: HE_R08 -> GND
- AMR1 pad 8: GND -> HE_R08
Routing:
- net HE_R07: track 127.4 -> 182.7 mm, vias 2 -> 6
- net HE_R05: track 54.1 -> 103.0 mm, vias 2 -> 10
- net MUX_A0: track 254.2 -> 298.0 mm, vias 9 -> 11
- net RGB_R_21: track 100.5 -> 58.2 mm, vias 6 -> 4
- net RGB_R_17: track 55.1 -> 21.5 mm, vias 4 -> 2
- net MUX_A2: track 184.2 -> 206.8 mm, vias 7 -> 13
- net HE_R20: track 72.4 -> 94.3 mm, vias 2 -> 10
- net +3V3A: track 1042.2 -> 1062.5 mm, vias 27 -> 37
- net HE_R08: track 93.9 -> 111.7 mm, vias 2 -> 6
- net HE_R11: track 19.3 -> 36.9 mm, vias 1 -> 2
- net MUX_A1: track 176.4 -> 192.3 mm
- net ADC_R3: track 79.0 -> 93.5 mm, vias 2 -> 6
- net HE_R06: track 101.9 -> 115.5 mm, vias 2 -> 8
- net ADC_R1: track 111.7 -> 121.8 mm
- net HE_R28: track 28.3 -> 37.3 mm, vias 0 -> 2
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