File: release/pcbway-pogo-neo/individual-boards/Controller/source/Symm60HE-Neo-Controller.kicad_pcb (KiCad board)
At the start: 2 copper layers, 57 x 27 mm, 38 parts, among them J1 TYPE-C-31-M-12, J2 FFC_12P, J3 FFC_12P, SW1 TS-1187A, SW2 TS-1187A, U1 AT32F405RCT7, U2 USBLC6-2SC6, U3 TLV75733PDBV, U4 XC6206P332MR, Y1 12MHz

Commit message: Replace the project with the reorganised T7 tree: ribbon keyboard is production, pogo archived
Production design is now the outward-facing FPC keyboard with per-key
SK6812MINI-E reverse-mount LEDs, a fifth SN74LV4051A mux per half so every
alternate Hall position has its own channel, an SN74AHCT1G125 LED level
shifter, a 50 x 31 mm daughterboard, 1.5 mm POM plates and 3 degree / 7 degree
tent and typing angles. The universal half panel is fully populated (359
placements) with routed NPTH alignment slots for the mutually exclusive
positions, and eight fixed-layout Left/Right PCB pairs are released under
release/layout-pcbs/ with matching BOM, CPL, Gerber ZIP, drill report and DRC.

Reorganise tools/ into cad/, generators/, layouts/, pcb/, pogo/, releases/ and
rendering/ subpackages; add designs/ and layout/ (KLE) trees and per-layout
gallery renders. The Fusion handoff is a fourteen-body reference STEP with
Gateron KS-20 switch and Cherry-profile keycap references and exact BOOMELE,
HRO and XKB models under case/fusion360/models/official/ with provenance.

The Neo-style pogo variant, its Mill-Max vendor models, the Fusion setup
script and the pogo release packages are archived as design history and
marked DO-NOT-ORDER. Their restored BOM snapshots had reintroduced the wrong
mux part C7792; corrected to C128414 / SN74LV4051ADR and their checksum lists
and archives rebuilt.

Co-Authored-By: Claude Opus 5 <noreply@anthropic.com>
Other:
- board size 57 x 27 mm -> 57 x 28 mm
Changed lines of the file:
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@@
 	)
 	(gr_line
-		(start 154.709 -5.7633)
+		(start 154.709 -6.7633)
 		(end 154.709 19.2367)
 		(stroke
@@
 	)
 	(gr_line
-		(start 154.7138 -5.8613)
-		(end 154.709 -5.7633)
+		(start 154.7138 -6.8613)
+		(end 154.709 -6.7633)
 		(stroke
 			(width 0.1)
@@
 	)
 	(gr_line
-		(start 154.7282 -5.9584)
-		(end 154.7138 -5.8613)
+		(start 154.7282 -6.9584)
+		(end 154.7138 -6.8613)
 		(stroke
 			(width 0.1)
@@
 	)
 	(gr_line
-		(start 154.7521 -6.0535)
-		(end 154.7282 -5.9584)
+		(start 154.7521 -7.0535)
+		(end 154.7282 -6.9584)
 		(stroke
 			(width 0.1)
@@
 	)
 	(gr_line
-		(start 154.7851 -6.1459)
-		(end 154.7521 -6.0535)
+		(start 154.7851 -7.1459)
+		(end 154.7521 -7.0535)
 		(stroke
 			(width 0.1)
@@
 	)
 	(gr_line
-		(start 154.8271 -6.2347)
-		(end 154.7851 -6.1459)
+		(start 154.8271 -7.2347)
+		(end 154.7851 -7.1459)
 		(stroke
 			(width 0.1)
@@
 	)
 	(gr_line
-		(start 154.8775 -6.3188)
-		(end 154.8271 -6.2347)
+		(start 154.8775 -7.3188)
+		(end 154.8271 -7.2347)
 		(stroke
 			(width 0.1)
@@
 	)
 	(gr_line
-		(start 154.936 -6.3977)
-		(end 154.8775 -6.3188)
+		(start 154.936 -7.3977)
+		(end 154.8775 -7.3188)
 		(stroke
 			(width 0.1)
@@
 	)
 	(gr_line
-		(start 155.0019 -6.4704)
-		(end 154.936 -6.3977)
+		(start 155.0019 -7.4704)
+		(end 154.936 -7.3977)
 		(stroke
 			(width 0.1)
@@
 	)
 	(gr_line
-		(start 155.0746 -6.5363)
-		(end 155.0019 -6.4704)
+		(start 155.0746 -7.5363)
+		(end 155.0019 -7.4704)
 		(stroke
 			(width 0.1)
@@
 	)
 	(gr_line
-		(start 155.1534 -6.5947)
-		(end 155.0746 -6.5363)
+		(start 155.1534 -7.5947)
+		(end 155.0746 -7.5363)
 		(stroke
 			(width 0.1)
@@
 	)
 	(gr_line
-		(start 155.2376 -6.6452)
-		(end 155.1534 -6.5947)
+		(start 155.2376 -7.6452)
+		(end 155.1534 -7.5947)
 		(stroke
 			(width 0.1)
@@
 	)
 	(gr_line
-		(start 155.3263 -6.6871)
-		(end 155.2376 -6.6452)
+		(start 155.3263 -7.6871)
+		(end 155.2376 -7.6452)
 		(stroke
 			(width 0.1)
@@
 	)
 	(gr_line
-		(start 155.4187 -6.7202)
-		(end 155.3263 -6.6871)
+		(start 155.4187 -7.7202)
+		(end 155.3263 -7.6871)
 		(stroke
 			(width 0.1)
@@
 	)
 	(gr_line
-		(start 155.5139 -6.744)
-		(end 155.4187 -6.7202)
+		(start 155.5139 -7.744)
+		(end 155.4187 -7.7202)
 		(stroke
 			(width 0.1)
@@
 	)
 	(gr_line
-		(start 155.611 -6.7584)
-		(end 155.5139 -6.744)
+		(start 155.611 -7.7584)
+		(end 155.5139 -7.744)
 		(stroke
 			(width 0.1)
@@
 	)
 	(gr_line
-		(start 155.709 -6.7633)
-		(end 155.611 -6.7584)
+		(start 155.709 -7.7633)
+		(end 155.611 -7.7584)
 		(stroke
 			(width 0.1)
@@
 	)
 	(gr_line
-		(start 210.709 -6.7633)
-		(end 155.709 -6.7633)
+		(start 210.709 -7.7633)
+		(end 155.709 -7.7633)
 		(stroke
 			(width 0.1)
@@
 	)
 	(gr_line
-		(start 210.807 -6.7584)
-		(end 210.709 -6.7633)
+		(start 210.807 -7.7584)
+		(end 210.709 -7.7633)
 		(stroke
 			(width 0.1)
@@
 	)
 	(gr_line
-		(start 210.9041 -6.744)
-		(end 210.807 -6.7584)
+		(start 210.9041 -7.744)
+		(end 210.807 -7.7584)
 		(stroke
 			(width 0.1)
@@
 	)
 	(gr_line
-		(start 210.9993 -6.7202)
-		(end 210.9041 -6.744)
+		(start 210.9993 -7.7202)
+		(end 210.9041 -7.744)
 		(stroke
 			(width 0.1)
@@
 	)
 	(gr_line
-		(start 211.0917 -6.6871)
-		(end 210.9993 -6.7202)
+		(start 211.0917 -7.6871)
+		(end 210.9993 -7.7202)
 		(stroke
 			(width 0.1)
@@
 	)
 	(gr_line
-		(start 211.1804 -6.6452)
-		(end 211.0917 -6.6871)
+		(start 211.1804 -7.6452)
+		(end 211.0917 -7.6871)
 		(stroke
 			(width 0.1)
@@
 	)
 	(gr_line
-		(start 211.2646 -6.5947)
-		(end 211.1804 -6.6452)
+		(start 211.2646 -7.5947)
+		(end 211.1804 -7.6452)
 		(stroke
 			(width 0.1)
@@
 	)
 	(gr_line
-		(start 211.3434 -6.5363)
-		(end 211.2646 -6.5947)
+		(start 211.3434 -7.5363)
+		(end 211.2646 -7.5947)
 		(stroke
 			(width 0.1)
@@
 	)
 	(gr_line
-		(start 211.4161 -6.4704)
-		(end 211.3434 -6.5363)
+		(start 211.4161 -7.4704)
+		(end 211.3434 -7.5363)
 		(stroke
 			(width 0.1)
@@
 	)
 	(gr_line
-		(start 211.482 -6.3977)
-		(end 211.4161 -6.4704)
+		(start 211.482 -7.3977)
+		(end 211.4161 -7.4704)
 		(stroke
 			(width 0.1)
@@
 	)
 	(gr_line
-		(start 211.5405 -6.3188)
-		(end 211.482 -6.3977)
+		(start 211.5405 -7.3188)
+		(end 211.482 -7.3977)
 		(stroke
 			(width 0.1)
@@
 	)
 	(gr_line
-		(start 211.5909 -6.2347)
-		(end 211.5405 -6.3188)
+		(start 211.5909 -7.2347)
+		(end 211.5405 -7.3188)
 		(stroke
 			(width 0.1)
@@
 	)
 	(gr_line
-		(start 211.6329 -6.1459)
-		(end 211.5909 -6.2347)
+		(start 211.6329 -7.1459)
+		(end 211.5909 -7.2347)
 		(stroke
 			(width 0.1)
@@
 	)
 	(gr_line
-		(start 211.6659 -6.0535)
-		(end 211.6329 -6.1459)
+		(start 211.6659 -7.0535)
+		(end 211.6329 -7.1459)
 		(stroke
 			(width 0.1)
@@
 	)
 	(gr_line
-		(start 211.6898 -5.9584)
-		(end 211.6659 -6.0535)
+		(start 211.6898 -6.9584)
+		(end 211.6659 -7.0535)
 		(stroke
 			(width 0.1)
@@
 	)
 	(gr_line
-		(start 211.7042 -5.8613)
-		(end 211.6898 -5.9584)
+		(start 211.7042 -6.8613)
+		(end 211.6898 -6.9584)
 		(stroke
 			(width 0.1)
@@
 	)
 	(gr_line
-		(start 211.709 -5.7633)
-		(end 211.7042 -5.8613)
+		(start 211.709 -6.7633)
+		(end 211.7042 -6.8613)
 		(stroke
 			(width 0.1)
@@
 	(gr_line
 		(start 211.709 19.2367)
-		(end 211.709 -5.7633)
-		(stroke
-			(width 0.1)
+		(end 211.709 -6.7633)
+		(stroke
+			(width 0.1)
