File: pcb/variants/layouts/wkl/Symm60HE-wkl-Left.kicad_pcb (KiCad board)
At the start: 2 copper layers, 145.9 x 104.7 mm, 168 parts

Commit message: Publish routed WKL PCBs and remove unrouted starters
Parts:
- RBPL29: footprint Symm60HE_Project:R3_R_0402_1005Metric -> Symm60HE_Project:R3_R_0402_1005Metric_DNP
- moved CML3 5.30 mm to (74.0, 57.6)
- moved CL16A 2.81 mm to (40.5, 39.5)
- moved CL17B 1.88 mm to (72.5, 54.3)
- moved MHL3 1.28 mm to (136.0, 49.2)
Routing:
- net HE_L24: track 39.8 -> 64.2 mm, vias 2 -> 4
- net +3V3A: track 1044.6 -> 1057.4 mm, vias 21 -> 23
- net HE_L20: track 74.6 -> 66.0 mm, vias 2 -> 4
- net RGB_L_09: track 31.9 -> 35.6 mm
- net RGB_L_17: track 30.4 -> 33.4 mm
- net HE_L17: track 18.5 -> 21.0 mm
- net VBUS: track 823.2 -> 825.4 mm
- net RGB_L_27: track 52.4 -> 54.5 mm
- net HE_L33: track 90.0 -> 92.0 mm, vias 5 -> 4
- net RGB_L_03: track 23.6 -> 25.3 mm
- net HE_L18: track 31.8 -> 33.1 mm
- net HE_L32: track 52.8 -> 53.9 mm
- net RGB_L_08: track 43.9 -> 45.0 mm
- net HE_L19: track 48.3 -> 47.7 mm
- net GND: vias 227 -> 96

Commit message: Publish 2026-10-05 production PCBs and firmware
Parts:
- AML1, AML2, AML3, AML4, AML5: footprint Symm60HE_Project:AM1_SOIC-16_3.9x9.9mm_P1.27mm -> Symm60HE_Project:AM1_TSSOP-16_4.4x5mm_P0.65mm
- moved AML5 76.0 mm to (75.4, 80.4)
- moved AML2 64.0 mm to (95.0, 24.5)
- moved AML1 56.0 mm to (82.0, 22.0)
- moved AML4 27.6 mm to (95.0, 63.0), turned to 90 degrees
- moved CRGBL13 5.85 mm to (110.0, 46.0)
- moved CRGBL16 4.42 mm to (105.0, 61.5)
- moved CL26A 3.84 mm to (116.0, 64.0)
- moved CL18A 3.39 mm to (74.8, 40.0)
- moved CL4B 3.00 mm to (77.2, 14.0)
- moved CL13B 2.94 mm to (124.0, 40.0)
- moved CL19B 2.94 mm to (107.7, 56.0)
- moved CL19A 2.75 mm to (96.8, 46.0)
- moved CL13A 2.36 mm to (111.0, 24.0)
- moved CML3 2.08 mm to (74.0, 55.5), turned to 0 degrees
- moved CRGBL4 1.59 mm to (70.5, 20.3)
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Connections:
- AML1 pad 1: HE_L05 -> HE_L11
- AML1 pad 12: HE_L04 -> HE_L01
- AML1 pad 13: HE_L01 -> HE_L02
- AML1 pad 14: HE_L02 -> HE_L03
- AML1 pad 15: HE_L03 -> HE_L04
- AML1 pad 2: HE_L07 -> HE_L10
- AML1 pad 4: HE_L08 -> HE_L09
- AML1 pad 5: HE_L06 -> HE_L08
- AML2 pad 1: HE_L13 -> HE_L14
- AML2 pad 12: HE_L12 -> HE_L05
- AML2 pad 13: HE_L09 -> HE_L06
- AML2 pad 14: HE_L10 -> HE_L07
- AML2 pad 15: HE_L11 -> (no net)
- AML2 pad 2: HE_L15 -> HE_L13
- AML2 pad 4: HE_L16 -> GND
- AML2 pad 5: HE_L14 -> HE_L12
- AML3 pad 1: HE_L21 -> HE_L24
- AML3 pad 12: HE_L20 -> HE_L15
- AML3 pad 13: HE_L17 -> HE_L16
- AML3 pad 14: HE_L18 -> HE_L17
- AML3 pad 15: HE_L19 -> HE_L18
- AML3 pad 4: HE_L24 -> HE_L22
- AML3 pad 5: HE_L22 -> HE_L21
- AML4 pad 1: HE_L29 -> HE_L26
- AML4 pad 12: HE_L28 -> HE_L19
- AML4 pad 13: HE_L25 -> GND
- AML4 pad 14: HE_L26 -> GND
- AML4 pad 15: HE_L27 -> HE_L20
- AML4 pad 2: HE_L31 -> GND
- AML4 pad 5: HE_L30 -> HE_L25
- AML5 pad 1: GND -> HE_L31
- AML5 pad 13: HE_L32 -> GND
- AML5 pad 14: HE_L33 -> GND
- AML5 pad 2: GND -> HE_L30
- AML5 pad 4: GND -> HE_L32
- AML5 pad 5: GND -> HE_L33
Routing:
- net VBUS: track 825.4 -> 1133.2 mm, vias 4 -> 58
- net +3V3A: track 1057.4 -> 1362.9 mm, vias 23 -> 65
- net ADC_L5: track 218.3 -> 75.5 mm
- net HE_L05: track 152.0 -> 12.2 mm, vias 2 -> 0
- net HE_L06: track 146.2 -> 43.9 mm, vias 2 -> 0
- net HE_L07: track 137.5 -> 63.7 mm, vias 2 -> 0
- net HE_L12: track 89.0 -> 16.0 mm, vias 2 -> 0
- net HE_L04: track 76.3 -> 16.1 mm, vias 2 -> 0
- net HE_L14: track 117.9 -> 58.8 mm, vias 2 -> 0
- net HE_L13: track 100.4 -> 50.6 mm, vias 2 -> 0
- net HE_L11: track 61.1 -> 15.8 mm, vias 2 -> 0
- net HE_L25: track 64.7 -> 20.7 mm, vias 2 -> 0
- net HE_L33: track 92.0 -> 50.1 mm, vias 4 -> 0
- net ADC_L2: track 111.8 -> 72.4 mm, vias 2 -> 4
- net GND: track 45.6 -> 6.59 mm, vias 96 -> 90
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