File: pcb/variants/layouts/wkl-left-arrows-right-bs2/Symm60HE-wkl-left-arrows-right-bs2-Right.kicad_pcb (KiCad board)
At the start: 2 copper layers, 145.9 x 104.7 mm, 175 parts

Commit message: Publish 2026-10-05 production PCBs and firmware
Parts:
- AMR1, AMR2, AMR3, AMR4, AMR5: footprint Symm60HE_Project:AM1_SOIC-16_3.9x9.9mm_P1.27mm -> Symm60HE_Project:AM1_TSSOP-16_4.4x5mm_P0.65mm
- RBPR24, RBPR31, RBPR5: footprint Symm60HE_Project:R3_R_0402_1005Metric -> Symm60HE_Project:R3_R_0402_1005Metric_DNP
- moved AMR5 76.4 mm to (226.6, 80.4), turned to 90 degrees
- moved AMR2 64.4 mm to (207.0, 24.5), turned to 90 degrees
- moved AMR1 44.2 mm to (235.0, 21.0), turned to 90 degrees
- moved AMR4 27.9 mm to (207.0, 63.0)
- moved CR16A 16.3 mm to (245.5, 48.6)
- moved CR8A 12.4 mm to (177.1, 18.1), turned to 9 degrees
- moved CR7A 12.3 mm to (195.9, 15.0), turned to 9 degrees
- moved CR14A 12.1 mm to (188.6, 35.0), turned to 9 degrees
- moved CR20A 12.1 mm to (202.8, 51.9), turned to 9 degrees
- moved CR21A 12.1 mm to (183.9, 54.9), turned to 9 degrees
- moved CR28A 12.1 mm to (199.3, 71.9), turned to 9 degrees
- moved CR29A 12.1 mm to (180.5, 74.9), turned to 9 degrees
- moved CR15A 12.1 mm to (169.7, 38.0), turned to 9 degrees
- moved CR6A 12.1 mm to (214.6, 12.3), turned to 6 degrees
- moved CR35A 12.1 mm to (219.8, 88.3), turned to 6 degrees
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Connections:
- AMR1 pad 1: HE_R05 -> HE_R12
- AMR1 pad 12: HE_R04 -> HE_R02
- AMR1 pad 13: HE_R01 -> HE_R03
- AMR1 pad 14: HE_R02 -> HE_R04
- AMR1 pad 15: HE_R03 -> GND
- AMR1 pad 2: HE_R07 -> HE_R11
- AMR1 pad 4: HE_R08 -> HE_R10
- AMR1 pad 5: HE_R06 -> HE_R09
- AMR2 pad 1: HE_R13 -> GND
- AMR2 pad 12: HE_R12 -> HE_R07
- AMR2 pad 13: HE_R09 -> HE_R06
- AMR2 pad 14: HE_R10 -> HE_R01
- AMR2 pad 15: HE_R11 -> GND
- AMR2 pad 2: HE_R15 -> HE_R08
- AMR2 pad 4: HE_R16 -> HE_R13
- AMR3 pad 1: HE_R21 -> HE_R25
- AMR3 pad 12: HE_R20 -> HE_R15
- AMR3 pad 13: HE_R17 -> HE_R16
- AMR3 pad 14: HE_R18 -> HE_R17
- AMR3 pad 15: HE_R19 -> HE_R18
- AMR3 pad 4: HE_R24 -> HE_R22
- AMR3 pad 5: HE_R22 -> HE_R21
- AMR4 pad 1: HE_R29 -> HE_R30
- AMR4 pad 12: HE_R28 -> HE_R20
- AMR4 pad 13: HE_R25 -> HE_R19
- AMR4 pad 14: HE_R26 -> GND
- AMR4 pad 15: HE_R27 -> GND
- AMR4 pad 2: HE_R31 -> HE_R34
- AMR4 pad 4: HE_R32 -> HE_R26
- AMR4 pad 5: HE_R30 -> HE_R27
- AMR5 pad 1: GND -> HE_R36
- AMR5 pad 12: HE_R36 -> GND
- AMR5 pad 13: HE_R33 -> GND
- AMR5 pad 14: HE_R34 -> GND
- AMR5 pad 15: HE_R35 -> GND
- AMR5 pad 2: GND -> HE_R35
- AMR5 pad 4: GND -> HE_R28
- AMR5 pad 5: GND -> HE_R32
- CR24B pad 1: HE_R24 -> HE_R25
- CR30B pad 1: HE_R29 -> HE_R35
- CR34B pad 1: HE_R31 -> HE_R36
- CR4B pad 1: HE_R33 -> HE_R04
- HER24 pad 3: HE_R24 -> HE_R25
- HER30 pad 3: HE_R29 -> HE_R35
- HER34 pad 3: HE_R31 -> HE_R36
- HER4 pad 3: HE_R33 -> HE_R04
Routing:
- net GND: track 212.8 -> 3.60 mm, vias 268 -> 161
- net VBUS: track 774.9 -> 964.1 mm, vias 15 -> 64
- net +3V3A: track 991.1 -> 1169.6 mm, vias 27 -> 89
- net HE_R08: track 110.5 -> 12.0 mm, vias 4 -> 0
- net HE_R02: track 105.1 -> 18.4 mm, vias 6 -> 2
- net HE_R07: track 127.4 -> 42.0 mm, vias 2 -> 0
- net ADC_R2: track 148.9 -> 64.9 mm
- net HE_R24: track 79.5 -> 0.00 mm, vias 7 -> 0
- net HE_R34: track 29.5 -> 109.0 mm, vias 0 -> 9
- net HE_R31: track 79.1 -> 0.00 mm, vias 4 -> 0
- net HE_R06: track 101.9 -> 22.9 mm, vias 2 -> 0
- net HE_R01: track 102.4 -> 25.8 mm, vias 6 -> 0
- net HE_R36: track 0.00 -> 74.9 mm, vias 0 -> 2
- net RGB_R_20: track 195.0 -> 121.3 mm, vias 4 -> 6
- net ADC_R5: track 152.4 -> 81.6 mm, vias 2 -> 0
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